Commit message: modify description; fix docker to download dependencies

File: my_diffbot_description/urdf/my_diffbot_description.xacro (robot description, xacro)
@@ -33,5 +33,4 @@
         <cylinder radius="0.15" length="0.06"/>
       </geometry>
-      <material name="orange"/>
     </visual>
     <inertial>
@@ -56,5 +55,4 @@
           <cylinder length="0.05" radius="0.025"/>
         </geometry>
-        <material name="blue"/>
       </visual>
     </link>
@@ -71,5 +69,4 @@
           <cylinder length="0.01" radius="0.015"/>
         </geometry>
-        <material name="blue"/>
       </visual>
     </link>
@@ -96,5 +93,4 @@
           <cylinder length="${wheel_len}" radius="${wheel_radius}"/>
         </geometry>
-        <material name="blue"/>
       </visual>
       <inertial>
@@ -128,5 +124,4 @@
           <cylinder length="${wheel_len}" radius="${wheel_radius}"/>
         </geometry>
-        <material name="blue"/>
       </visual>
       <inertial>
@@ -157,5 +152,4 @@
           <sphere radius="${caster_wheel_radius}"/>
         </geometry>
-        <material name="white"/>
       </visual>
       <inertial>
@@ -186,5 +180,4 @@
           <sphere radius="${caster_wheel_radius}"/>
         </geometry>
-        <material name="white"/>
       </visual>
       <inertial>

Commit message: hotfix(description): fix lidar orientation

File: my_diffbot_description/urdf/my_diffbot_description.xacro (robot description, xacro)
@@ -47,5 +47,5 @@
       <parent link="${prefix}base_link"/>
       <child link="${prefix}lidar_link"/>
-      <origin xyz="0.06 0.06 0.15" rpy="0.0 0.0 0.0"/>
+      <origin xyz="0.06 0.06 0.15" rpy="0.0 0.0 -1.57"/>
     </joint>
     <link name="${prefix}lidar_link">

Commit message: Update description

File: my_diffbot_description/urdf/my_diffbot_description.xacro (robot description, xacro)
@@ -47,5 +47,5 @@
       <parent link="${prefix}base_link"/>
       <child link="${prefix}lidar_link"/>
-      <origin xyz="0.06 0.06 0.15" rpy="0.0 0.0 -1.57"/>
+      <origin xyz="0.06 0.01 0.10" rpy="0.0 0.0 -1.57"/>
     </joint>
     <link name="${prefix}lidar_link">
@@ -61,5 +61,5 @@
       <parent link="${prefix}base_link"/>
       <child link="${prefix}imu_link"/>
-      <origin xyz="-0.04 -0.06 0.05" rpy="0.0 0.0 0.0"/>
+      <origin xyz="0.0 -0.015 0.065" rpy="0.0 0.0 0.0"/>
     </joint>
     <link name="${prefix}imu_link">

Commit message: Update description

File: my_diffbot_description/urdf/my_diffbot_description.xacro (robot description, xacro)
@@ -61,5 +61,5 @@
       <parent link="${prefix}base_link"/>
       <child link="${prefix}imu_link"/>
-      <origin xyz="0.0 -0.015 0.065" rpy="0.0 0.0 0.0"/>
+      <origin xyz="0.0 0.025 0.065" rpy="0.0 0.0 0.0"/>
     </joint>
     <link name="${prefix}imu_link">

Commit message: Add BNO055 IMU (#2)

File: my_diffbot_description/urdf/my_diffbot_description.xacro (robot description, xacro)
@@ -47,5 +47,5 @@
       <parent link="${prefix}base_link"/>
       <child link="${prefix}lidar_link"/>
-      <origin xyz="0.06 0.06 0.15" rpy="0.0 0.0 -1.57"/>
+      <origin xyz="0.06 0.01 0.10" rpy="0.0 0.0 -1.57"/>
     </joint>
     <link name="${prefix}lidar_link">
@@ -61,5 +61,5 @@
       <parent link="${prefix}base_link"/>
       <child link="${prefix}imu_link"/>
-      <origin xyz="-0.04 -0.06 0.05" rpy="0.0 0.0 0.0"/>
+      <origin xyz="0.0 0.025 0.065" rpy="0.0 0.0 0.0"/>
     </joint>
     <link name="${prefix}imu_link">

Commit message: Add ultrasonic sensor

File: my_diffbot_description/urdf/my_diffbot_description.xacro (robot description, xacro)
@@ -57,4 +57,18 @@
       </visual>
     </link>
+    <!-- Ultrasonic -->
+    <joint name="ultrasonic_joint" type="fixed">
+      <parent link="${prefix}base_link"/>
+      <child link="${prefix}Ultrasonic_link"/>
+      <origin xyz="-0.12 0.0 0.0" rpy="0.0 0.0 -3.14"/>
+    </joint>
+    <link name="${prefix}Ultrasonic_link">
+      <visual>
+        <origin xyz="0 0 0" rpy="0 0 0"/>
+        <geometry>
+          <cylinder length="0.01" radius="0.015"/>
+        </geometry>
+      </visual>
+    </link>
     <!-- IMU -->
     <joint name="imu_joint" type="fixed">

File: my_diffbot_description/urdf/my_diffbot_ros2_control.xacro (robot description, xacro)
@@ -40,4 +40,7 @@
         <state_interface name="velocity"/>
       </joint>
+      <sensor name="ultrasonic_sensor">
+        <state_interface name="range"/>
+      </sensor>
     </ros2_control>
   </xacro:macro>

Commit message: Add launch

File: my_diffbot_description/urdf/my_diffbot_description.xacro (robot description, xacro)
@@ -60,8 +60,8 @@
     <joint name="ultrasonic_joint" type="fixed">
       <parent link="${prefix}base_link"/>
-      <child link="${prefix}Ultrasonic_link"/>
+      <child link="${prefix}ultrasonic_link"/>
       <origin xyz="-0.12 0.0 0.0" rpy="0.0 0.0 -3.14"/>
     </joint>
-    <link name="${prefix}Ultrasonic_link">
+    <link name="${prefix}ultrasonic_link">
       <visual>
         <origin xyz="0 0 0" rpy="0 0 0"/>

Commit message: feat(hwi): add ultrasonic sensor (#3)

File: my_diffbot_description/urdf/my_diffbot_description.xacro (robot description, xacro)
@@ -57,4 +57,18 @@
       </visual>
     </link>
+    <!-- Ultrasonic -->
+    <joint name="ultrasonic_joint" type="fixed">
+      <parent link="${prefix}base_link"/>
+      <child link="${prefix}ultrasonic_link"/>
+      <origin xyz="-0.12 0.0 0.0" rpy="0.0 0.0 -3.14"/>
+    </joint>
+    <link name="${prefix}ultrasonic_link">
+      <visual>
+        <origin xyz="0 0 0" rpy="0 0 0"/>
+        <geometry>
+          <cylinder length="0.01" radius="0.015"/>
+        </geometry>
+      </visual>
+    </link>
     <!-- IMU -->
     <joint name="imu_joint" type="fixed">

Commit message: hotfix(description): moved lidar

File: my_diffbot_description/urdf/my_diffbot_description.xacro (robot description, xacro)
@@ -47,5 +47,5 @@
       <parent link="${prefix}base_link"/>
       <child link="${prefix}lidar_link"/>
-      <origin xyz="0.06 0.01 0.10" rpy="0.0 0.0 -1.57"/>
+      <origin xyz="0.06 0.01 0.10" rpy="0.0 0.0 1.57"/>
     </joint>
     <link name="${prefix}lidar_link">

Commit message: Revert "hotfix(description): moved lidar"
This reverts commit f1657f42a3ea321087470a1e016ab1756416b602.

File: my_diffbot_description/urdf/my_diffbot_description.xacro (robot description, xacro)
@@ -47,5 +47,5 @@
       <parent link="${prefix}base_link"/>
       <child link="${prefix}lidar_link"/>
-      <origin xyz="0.06 0.01 0.10" rpy="0.0 0.0 1.57"/>
+      <origin xyz="0.06 0.01 0.10" rpy="0.0 0.0 -1.57"/>
     </joint>
     <link name="${prefix}lidar_link">

Commit message: Update lidar position

File: my_diffbot_description/urdf/my_diffbot_description.xacro (robot description, xacro)
@@ -47,5 +47,5 @@
       <parent link="${prefix}base_link"/>
       <child link="${prefix}lidar_link"/>
-      <origin xyz="0.06 0.01 0.10" rpy="0.0 0.0 -1.57"/>
+      <origin xyz="-0.06 0.0 0.14" rpy="0.0 0.0 -1.57"/>
     </joint>
     <link name="${prefix}lidar_link">

Commit message: update joint velocity limit

File: my_diffbot_description/urdf/my_diffbot_description.xacro (robot description, xacro)
@@ -92,5 +92,5 @@
       <axis xyz="0 1 0"/>
       <dynamics damping="0.2"/>
-      <limit effort="100" velocity="1.0"/>
+      <limit effort="100" velocity="16.0"/>
     </joint>
     <!-- left wheel Link -->
@@ -123,5 +123,5 @@
       <axis xyz="0 1 0"/>
       <dynamics damping="0.2"/>
-      <limit effort="100" velocity="1.0"/>
+      <limit effort="100" velocity="16.0"/>
     </joint>
     <!-- right wheel Link -->

Commit message: hotfix

File: my_diffbot_description/urdf/my_diffbot_description.xacro (robot description, xacro)
@@ -47,5 +47,5 @@
       <parent link="${prefix}base_link"/>
       <child link="${prefix}lidar_link"/>
-      <origin xyz="-0.06 0.0 0.14" rpy="0.0 0.0 -1.57"/>
+      <origin xyz="-0.06 0.0 0.14" rpy="0.0 0.0 1.57"/>
     </joint>
     <link name="${prefix}lidar_link">

Commit message: hotfix(description): update base width

File: my_diffbot_description/urdf/my_diffbot_description.xacro (robot description, xacro)
@@ -5,5 +5,5 @@
   <xacro:property name="PI" value="3.1415926535897931"/>
   <xacro:property name="base_mass" value="0.3" /> <!-- arbitrary value for base mass -->
-  <xacro:property name="base_width" value="0.2" />
+  <xacro:property name="base_width" value="0.28" />
   <xacro:property name="base_length" value="0.3" />
   <xacro:property name="base_height" value="0.06" />
