Commit message: update description

File: my_diffbot_description/urdf/my_diffbot_description.xacro (robot description, xacro)
@@ -48,5 +48,5 @@
       <parent link="${prefix}base_link"/>
       <child link="${prefix}lidar_link"/>
-      <origin xyz="-0.06 0.0 0.14" rpy="0.0 0.0 1.57"/>
+      <origin xyz="0.10 -0.02 0.14" rpy="0.0 0.0 -1.57"/>
     </joint>
     <link name="${prefix}lidar_link">
@@ -76,5 +76,5 @@
       <parent link="${prefix}base_link"/>
       <child link="${prefix}imu_link"/>
-      <origin xyz="0.0 0.025 0.065" rpy="0.0 0.0 0.0"/>
+      <origin xyz="0.04 0.0 0.045" rpy="0.0 0.0 0.0"/>
     </joint>
     <link name="${prefix}imu_link">
