Commit message: fix(description): raise wheel joint velocity limit to 40 rad/s
Previous limit of 16 rad/s was being exceeded by diff_drive commands
(~16.13 rad/s), causing throttled controller_manager errors.

Co-Authored-By: Claude Sonnet 4.6 <noreply@anthropic.com>

File: my_diffbot_description/urdf/my_diffbot_description.xacro (robot description, xacro)
@@ -92,5 +92,5 @@
       <axis xyz="0 1 0"/>
       <dynamics damping="0.2"/>
-      <limit effort="100" velocity="16.0"/>
+      <limit effort="100" velocity="40.0"/>
     </joint>
     <!-- left wheel Link -->
@@ -123,5 +123,5 @@
       <axis xyz="0 1 0"/>
       <dynamics damping="0.2"/>
-      <limit effort="100" velocity="16.0"/>
+      <limit effort="100" velocity="40.0"/>
     </joint>
     <!-- right wheel Link -->

File: my_diffbot_description/urdf/my_diffbot_ros2_control.xacro (robot description, xacro)
@@ -28,6 +28,6 @@
       <joint name="right_wheel_joint">
         <command_interface name="velocity">
-          <param name="min">-16.00</param>
-          <param name="max">16.00</param>
+          <param name="min">-40.00</param>
+          <param name="max">40.00</param>
         </command_interface>
         <state_interface name="position"/>
@@ -36,6 +36,6 @@
       <joint name="left_wheel_joint">
         <command_interface name="velocity">
-          <param name="min">-16.00</param>
-          <param name="max">16.00</param>
+          <param name="min">-40.00</param>
+          <param name="max">40.00</param>
         </command_interface>
         <state_interface name="position"/>

Commit message: fix(description): use the measured wheel separation and radius
Remeasured on the robot: 0.23 m between the wheels and 6 cm wheel
diameter (was 0.285 m and 0.031 m). A commanded 1.5 rad/s spin now reads
1.50 rad/s on the IMU instead of 1.83. The URDF places the wheel joints
from a separate wheel_separation, since base_width also positions the
casters.

Co-Authored-By: Claude Opus 5.5 <noreply@anthropic.com>

File: my_diffbot_description/urdf/my_diffbot_description.xacro (robot description, xacro)
@@ -10,5 +10,6 @@
   <xacro:property name="wheel_mass" value="0.3" /> <!-- arbitrary value for wheel mass -->
   <xacro:property name="wheel_len" value="0.025" />
-  <xacro:property name="wheel_radius" value="0.031" />
+  <xacro:property name="wheel_radius" value="0.03" />
+  <xacro:property name="wheel_separation" value="0.23" />
   <xacro:property name="caster_wheel_mass" value="0.1" /> <!-- arbitrary value for caster wheel mass -->
   <xacro:property name="caster_wheel_radius" value="0.015" />
@@ -89,5 +90,5 @@
       <parent link="${prefix}base_link"/>
       <child link="${prefix}left_wheel"/>
-      <origin xyz="0 -${base_width/2} ${z_offset}" rpy="0 0 0"/>
+      <origin xyz="0 -${wheel_separation/2} ${z_offset}" rpy="0 0 0"/>
       <axis xyz="0 1 0"/>
       <dynamics damping="0.2"/>
@@ -120,5 +121,5 @@
       <parent link="${prefix}base_link"/>
       <child link="${prefix}right_wheel"/>
-      <origin xyz="0 ${base_width/2} ${z_offset}" rpy="0 0 0"/>
+      <origin xyz="0 ${wheel_separation/2} ${z_offset}" rpy="0 0 0"/>
       <axis xyz="0 1 0"/>
       <dynamics damping="0.2"/>

Commit message: fix(description): measure wheel separation centre to centre (0.255 m)
diff_drive needs the distance between the wheel contact centres; 0.23 m
was inner edge to inner edge, one 25 mm wheel width short. With 0.23
the wheel odometry over-reported rotation by 11-12 % against lidar scan
matching over ~360 deg spins; with 0.255 it is within +/-1.2 % (8 turns,
1.0 and 1.5 rad/s, both directions).

Co-Authored-By: Claude Opus 5.5 <noreply@anthropic.com>
Claude-Session: https://claude.ai/code/session_01WRYdMVDqFS9GLxapdNQxoF

File: my_diffbot_description/urdf/my_diffbot_description.xacro (robot description, xacro)
@@ -11,5 +11,5 @@
   <xacro:property name="wheel_len" value="0.025" />
   <xacro:property name="wheel_radius" value="0.03" />
-  <xacro:property name="wheel_separation" value="0.23" />
+  <xacro:property name="wheel_separation" value="0.255" />  <!-- wheel centre to centre -->
   <xacro:property name="caster_wheel_mass" value="0.1" /> <!-- arbitrary value for caster wheel mass -->
   <xacro:property name="caster_wheel_radius" value="0.015" />

Commit message: fix(description): match the lidar, IMU and wheel frames to the robot
Measured on the robot by driving 0.16 m straights and +/-90 deg turns and
fitting the lidar pose from scan matching against odom (three runs agree
within ~1 mm and 0.6 deg):

- lidar_link: x 0.110, y -0.023, yaw -1.510 (-86.5 deg, not -90). z 0.14
  is the hand measurement from the axle centre.
- imu_joint yaw = pi: /imu/data x points to the robot's rear (acceleration
  integrates to -v when driving forward). The EKF only fuses yaw and yaw
  rate, so this did not change its output, but x_accel or roll/pitch would
  have come out with the wrong sign.
- left_wheel sits at +y and right_wheel at -y (they were swapped).
- base_link is the axle centre, where the sensors were measured from:
  base_footprint -> base_link = wheel radius, so the wheels and casters
  touch the floor. The chassis and ultrasonic keep their physical place.

The README wheel numbers (31 mm / 160 mm) were stale: 30 mm / 255 mm.

Co-Authored-By: Claude Opus 5.5 <noreply@anthropic.com>
Claude-Session: https://claude.ai/code/session_014KtF8zZNgvjM3Zu3cmQvHV

File: my_diffbot_description/urdf/my_diffbot_description.xacro (robot description, xacro)
@@ -14,15 +14,15 @@
   <xacro:property name="caster_wheel_mass" value="0.1" /> <!-- arbitrary value for caster wheel mass -->
   <xacro:property name="caster_wheel_radius" value="0.015" />
-  <xacro:property name="z_offset" value="-${base_height/2}" /> <!-- Space btw top of beam and the each joint -->
-  <!-- Base Link -->
+  <xacro:property name="chassis_z" value="0.03" /> <!-- chassis bottom above the axle -->
+  <!-- Base Link: base_link is the axle centre, midway between the wheels -->
   <link name="base_footprint"/>
   <joint name="footprint_joint" type="fixed">
     <parent link="base_footprint"/>
     <child link="${prefix}base_link"/>
-    <origin xyz="0.0 0.0 0.05" rpy="0.0 0.0 0.0"/>
+    <origin xyz="0.0 0.0 ${wheel_radius}" rpy="0.0 0.0 0.0"/>
   </joint>
   <link name="${prefix}base_link">
     <collision>
-      <origin xyz="0 0 ${base_height/2}" rpy="0 0 0"/>
+      <origin xyz="0 0 ${chassis_z + base_height/2}" rpy="0 0 0"/>
       <geometry>
         <cylinder radius="0.15" length="0.06"/>
@@ -30,5 +30,5 @@
     </collision>
     <visual>
-      <origin xyz="0 0 ${base_height/2}" rpy="0 0 0"/>
+      <origin xyz="0 0 ${chassis_z + base_height/2}" rpy="0 0 0"/>
       <geometry>
         <cylinder radius="0.15" length="0.06"/>
@@ -36,5 +36,5 @@
     </visual>
     <inertial>
-      <origin xyz="0 0 0" rpy="0 0 0"/>
+      <origin xyz="0 0 ${chassis_z + base_height/2}" rpy="0 0 0"/>
       <mass value="${base_mass}"/>
       <inertia
@@ -44,9 +44,10 @@
       </inertial>
     </link>
-    <!-- LIDAR -->
+    <!-- LIDAR: x, y and yaw are the LD06 scan frame, fitted from scan matching over
+         straight drives and in-place turns (yaw -86.5 deg, not -90) -->
     <joint name="lidar_joint" type="fixed">
       <parent link="${prefix}base_link"/>
       <child link="${prefix}lidar_link"/>
-      <origin xyz="0.10 -0.02 0.14" rpy="0.0 0.0 -1.57"/>
+      <origin xyz="0.110 -0.023 0.14" rpy="0.0 0.0 -1.510"/>
     </joint>
     <link name="${prefix}lidar_link">
@@ -62,5 +63,5 @@
       <parent link="${prefix}base_link"/>
       <child link="${prefix}ultrasonic_link"/>
-      <origin xyz="-0.12 0.0 0.0" rpy="0.0 0.0 -3.14"/>
+      <origin xyz="-0.12 0.0 ${chassis_z}" rpy="0.0 0.0 -3.14"/>
     </joint>
     <link name="${prefix}ultrasonic_link">
@@ -72,9 +73,9 @@
       </visual>
     </link>
-    <!-- IMU -->
+    <!-- IMU: the firmware remap leaves /imu/data x pointing to the rear (accel while driving) -->
     <joint name="imu_joint" type="fixed">
       <parent link="${prefix}base_link"/>
       <child link="${prefix}imu_link"/>
-      <origin xyz="0.04 0.0 0.045" rpy="0.0 0.0 0.0"/>
+      <origin xyz="0.04 0.0 0.045" rpy="0.0 0.0 ${PI}"/>
     </joint>
     <link name="${prefix}imu_link">
@@ -90,5 +91,5 @@
       <parent link="${prefix}base_link"/>
       <child link="${prefix}left_wheel"/>
-      <origin xyz="0 -${wheel_separation/2} ${z_offset}" rpy="0 0 0"/>
+      <origin xyz="0 ${wheel_separation/2} 0" rpy="0 0 0"/>
       <axis xyz="0 1 0"/>
       <dynamics damping="0.2"/>
@@ -121,5 +122,5 @@
       <parent link="${prefix}base_link"/>
       <child link="${prefix}right_wheel"/>
-      <origin xyz="0 ${wheel_separation/2} ${z_offset}" rpy="0 0 0"/>
+      <origin xyz="0 -${wheel_separation/2} 0" rpy="0 0 0"/>
       <axis xyz="0 1 0"/>
       <dynamics damping="0.2"/>
@@ -152,5 +153,5 @@
       <parent link="${prefix}base_link"/>
       <child link="${prefix}caster_frontal_wheel"/>
-      <origin xyz="${base_width/2 - caster_wheel_radius} 0 ${z_offset}" rpy="0 0 0"/>
+      <origin xyz="${base_width/2 - caster_wheel_radius} 0 ${caster_wheel_radius - wheel_radius}" rpy="0 0 0"/>
     </joint>
     <!-- caster frontal wheel Link -->
@@ -180,5 +181,5 @@
       <parent link="${prefix}base_link"/>
       <child link="${prefix}caster_rear_wheel"/>
-      <origin xyz="${-base_width/2 + caster_wheel_radius} 0 ${z_offset}" rpy="0 0 0"/>
+      <origin xyz="${-base_width/2 + caster_wheel_radius} 0 ${caster_wheel_radius - wheel_radius}" rpy="0 0 0"/>
     </joint>
     <!-- caster rear wheel Link -->

Commit message: fix(description): add the 5.9 deg IMU board pitch to imu_joint
After a full BNO055 calibration (saved and restored by the firmware,
|a| 9.74 m/s2) the at-rest accel still reads +1.0 m/s2 along the IMU x
axis, while the 2 deg roll seen before calibration was bias. The lidar
plane is level within ~2 deg, so the tilt is the board's mount, not the
chassis. The 2D EKF ignores roll and pitch, so this only corrects TF.

Co-Authored-By: Claude Opus 5.5 <noreply@anthropic.com>
Claude-Session: https://claude.ai/code/session_014KtF8zZNgvjM3Zu3cmQvHV

File: my_diffbot_description/urdf/my_diffbot_description.xacro (robot description, xacro)
@@ -73,9 +73,10 @@
       </visual>
     </link>
-    <!-- IMU: the firmware remap leaves /imu/data x pointing to the rear (accel while driving) -->
+    <!-- IMU: the firmware remap leaves /imu/data x pointing to the rear (accel while driving).
+         The board is pitched 5.9 deg (calibrated accel at rest; the lidar plane is level). -->
     <joint name="imu_joint" type="fixed">
       <parent link="${prefix}base_link"/>
       <child link="${prefix}imu_link"/>
-      <origin xyz="0.04 0.0 0.045" rpy="0.0 0.0 ${PI}"/>
+      <origin xyz="0.04 0.0 0.045" rpy="0.0 -0.103 ${PI}"/>
     </joint>
     <link name="${prefix}imu_link">

Commit message: feat(description): reverse the base, sensors now at the rear
Rotate the lidar, IMU and ultrasonic mounts 180 deg about z
(x,y -> -x,-y, yaw + pi) so the old front is the new rear.

Co-Authored-By: Claude Opus 5.5 <noreply@anthropic.com>
Claude-Session: https://claude.ai/code/session_01UEzrzT2v2Gej1u4iKEhmYT

File: my_diffbot_description/urdf/my_diffbot_description.xacro (robot description, xacro)
@@ -45,9 +45,10 @@
     </link>
     <!-- LIDAR: x, y and yaw are the LD06 scan frame, fitted from scan matching over
-         straight drives and in-place turns (yaw -86.5 deg, not -90) -->
+         straight drives and in-place turns (yaw -86.5 deg, not -90), then rotated 180 deg
+         about z when the base was reversed (old front is now the rear) -->
     <joint name="lidar_joint" type="fixed">
       <parent link="${prefix}base_link"/>
       <child link="${prefix}lidar_link"/>
-      <origin xyz="0.110 -0.023 0.14" rpy="0.0 0.0 -1.510"/>
+      <origin xyz="-0.110 0.023 0.14" rpy="0.0 0.0 ${-1.510 + PI}"/>
     </joint>
     <link name="${prefix}lidar_link">
@@ -63,5 +64,5 @@
       <parent link="${prefix}base_link"/>
       <child link="${prefix}ultrasonic_link"/>
-      <origin xyz="-0.12 0.0 ${chassis_z}" rpy="0.0 0.0 -3.14"/>
+      <origin xyz="0.12 0.0 ${chassis_z}" rpy="0.0 0.0 0.0"/>
     </joint>
     <link name="${prefix}ultrasonic_link">
@@ -73,10 +74,11 @@
       </visual>
     </link>
-    <!-- IMU: the firmware remap leaves /imu/data x pointing to the rear (accel while driving).
+    <!-- IMU: the firmware remap leaves /imu/data x pointing to the old rear, which is the
+         front since the base was reversed (accel while driving).
          The board is pitched 5.9 deg (calibrated accel at rest; the lidar plane is level). -->
     <joint name="imu_joint" type="fixed">
       <parent link="${prefix}base_link"/>
       <child link="${prefix}imu_link"/>
-      <origin xyz="0.04 0.0 0.045" rpy="0.0 -0.103 ${PI}"/>
+      <origin xyz="-0.04 0.0 0.045" rpy="0.0 -0.103 0.0"/>
     </joint>
     <link name="${prefix}imu_link">
