Commit message: feat(hardware): run my_diffbot on the Kestrel ESP32-S3 base (#13)
* feat(hardware): drive the RoboAuto ESP32-S3 base over its binary protocol

Replace the ASCII serial MCU link with the RoboAuto binary protocol
(ported from cbot_hardware_interface, RoboAuto subset only): wheel
velocity commands, encoder position/velocity states, BNO055 IMU state
interfaces with /diagnostics, and led / roboauto_pid / roboauto_watchdog
gpios. The first WHEEL_FEEDBACK after activation only seeds the tick
baseline, since the firmware keeps counting across host reconnects.
Defaults: /dev/roboauto, CPR 515, kp=1 ki=3.

Co-Authored-By: Claude Opus 5.5 <noreply@anthropic.com>

* feat(bringup): publish the RoboAuto IMU and gpio controllers

Spawn imu_broadcaster (remapped to /imu/data, frame imu_link),
led_controller and roboauto_tuning_controller, and raise the controller
manager to 100 Hz to match the firmware's 50 Hz wheel / 100 Hz IMU
streams. The Jetson I2C bno055 node is gone; use_imu now only enables
the EKF.

Co-Authored-By: Claude Opus 5.5 <noreply@anthropic.com>

* chore(docker): swap the bno055 node deps for the RoboAuto controllers

Drop the bno055 repo, its pip packages and the I2C group; install
imu_sensor_broadcaster and gpio_controllers; mount the live /dev so
/dev/roboauto survives an ESP32 reset; add the 303a:4001 udev rule.

Co-Authored-By: Claude Opus 5.5 <noreply@anthropic.com>

* docs(readme): document the RoboAuto base, udev rules and gpio controllers

Co-Authored-By: Claude Opus 5.5 <noreply@anthropic.com>

* fix(hardware): report an identity IMU orientation until the first frame

A zero quaternion before the first IMU_DATA (or with no BNO055) would
put NaNs into the EKF, and the filter never recovers from them.

Co-Authored-By: Claude Opus 5.5 <noreply@anthropic.com>

* feat(bringup): always fuse the RoboAuto IMU through the EKF

Drop use_imu; the EKF always runs. diff_drive keeps its own odom topic
as the EKF input (it was remapped to /odom, leaving odom0 without a
publisher) and no longer broadcasts odom -> base_footprint, so the EKF
is the single owner of /odom and the odom TF.

Co-Authored-By: Claude Opus 5.5 <noreply@anthropic.com>

* feat(bringup): start the EKF from robot_controllers.launch.py

The EKF owns /odom and the odom TF, so it has to run whenever the
controllers do, including robot_controllers.launch.py on its own.
bringup_robot includes it through that file, so it still runs once.

Co-Authored-By: Claude Opus 5.5 <noreply@anthropic.com>

* fix(description): use the measured wheel separation and radius

Remeasured on the robot: 0.23 m between the wheels and 6 cm wheel
diameter (was 0.285 m and 0.031 m). A commanded 1.5 rad/s spin now reads
1.50 rad/s on the IMU instead of 1.83. The URDF places the wheel joints
from a separate wheel_separation, since base_width also positions the
casters.

Co-Authored-By: Claude Opus 5.5 <noreply@anthropic.com>

* feat(bringup): lower the base speed limit and ramp its acceleration

The RoboAuto wheels top out near 0.44 m/s on the floor, so cap linear
speed at 0.35 m/s to keep the wheel PID out of saturation. Stepped
setpoints wound up the firmware integrator behind its 100 ms speed
window and overshot by 22-26 %; ramping at 0.5 m/s^2 roughly halves
that. Deceleration is allowed to be faster than acceleration.

Co-Authored-By: Claude Opus 5.5 <noreply@anthropic.com>

* feat(hardware): default the wheel PID integral gain to 2

Floor step tests with ramped setpoints: ki=3 overshot 15-16 % on a
1000 mrps straight, ki=2 12.6 % and ki=1 10.7 %, while ki=1 doubled the
low-speed steady-state error. kp stays at 1.

Co-Authored-By: Claude Opus 5.5 <noreply@anthropic.com>

* fix(description): measure wheel separation centre to centre (0.255 m)

diff_drive needs the distance between the wheel contact centres; 0.23 m
was inner edge to inner edge, one 25 mm wheel width short. With 0.23
the wheel odometry over-reported rotation by 11-12 % against lidar scan
matching over ~360 deg spins; with 0.255 it is within +/-1.2 % (8 turns,
1.0 and 1.5 rad/s, both directions).

Co-Authored-By: Claude Opus 5.5 <noreply@anthropic.com>
Claude-Session: https://claude.ai/code/session_01WRYdMVDqFS9GLxapdNQxoF

* fix(localization): stop fusing the IMU x acceleration

The RoboAuto IMU_DATA acceleration includes gravity and the EKF does not
remove it, so any tilt leaks into x_accel as a velocity bias. Heading
stays on the BNO055 absolute yaw, which matched lidar scan matching
within +/-0.5 % per turn; its raw gyro reads ~3 % high.

Co-Authored-By: Claude Opus 5.5 <noreply@anthropic.com>
Claude-Session: https://claude.ai/code/session_01WRYdMVDqFS9GLxapdNQxoF

* set default port to /dev/ttyACM0

* update description

* fix(description): match the lidar, IMU and wheel frames to the robot

Measured on the robot by driving 0.16 m straights and +/-90 deg turns and
fitting the lidar pose from scan matching against odom (three runs agree
within ~1 mm and 0.6 deg):

- lidar_link: x 0.110, y -0.023, yaw -1.510 (-86.5 deg, not -90). z 0.14
  is the hand measurement from the axle centre.
- imu_joint yaw = pi: /imu/data x points to the robot's rear (acceleration
  integrates to -v when driving forward). The EKF only fuses yaw and yaw
  rate, so this did not change its output, but x_accel or roll/pitch would
  have come out with the wrong sign.
- left_wheel sits at +y and right_wheel at -y (they were swapped).
- base_link is the axle centre, where the sensors were measured from:
  base_footprint -> base_link = wheel radius, so the wheels and casters
  touch the floor. The chassis and ultrasonic keep their physical place.

The README wheel numbers (31 mm / 160 mm) were stale: 30 mm / 255 mm.

Co-Authored-By: Claude Opus 5.5 <noreply@anthropic.com>
Claude-Session: https://claude.ai/code/session_014KtF8zZNgvjM3Zu3cmQvHV

* fix(description): match the Gazebo model to the real robot

- DiffDrive: wheel separation 0.255 and radius 0.03 (was 0.21 / 0.0826),
  limits from base_controllers.yaml, and odom -> base_footprint, since
  base_link already has base_footprint as its parent.
- Lidar: LD06-like 360 deg, 455 beams, 0.02-12 m (was +/-80 deg, 10 m).
- Drop the depth camera: it referenced a camera_link that does not exist
  and the robot has no camera.
- Add the BNO055 as an IMU sensor on imu_link publishing imu/data, which
  the EKF fuses. It needs gz-sim-imu-system in the world.

Co-Authored-By: Claude Opus 5.5 <noreply@anthropic.com>
Claude-Session: https://claude.ai/code/session_014KtF8zZNgvjM3Zu3cmQvHV

* fix(bringup): fit the effective wheel radius and separation on the floor

Measured against lidar scan matching on the robot:
- wheel_radius 0.0308: four 1 m straight legs gave 0.03065-0.03091 (the
  wheel odometry under-reported distance by ~2.6 %).
- wheel_separation 0.250: four 720 deg in-place spins at 1 rad/s gave
  0.2494-0.2506 with that radius. Lidar and IMU yaw agreed within 0.1 %.
  With 0.255 / 0.03 the wheel odometry under-reported turning by ~4.5 %.

These are effective values (tyre contact, scrub, encoder); the URDF keeps
the physical 0.255 m centre to centre and 30 mm wheels.

Co-Authored-By: Claude Opus 5.5 <noreply@anthropic.com>
Claude-Session: https://claude.ai/code/session_014KtF8zZNgvjM3Zu3cmQvHV

* fix(description): add the 5.9 deg IMU board pitch to imu_joint

After a full BNO055 calibration (saved and restored by the firmware,
|a| 9.74 m/s2) the at-rest accel still reads +1.0 m/s2 along the IMU x
axis, while the 2 deg roll seen before calibration was bias. The lidar
plane is level within ~2 deg, so the tilt is the board's mount, not the
chassis. The 2D EKF ignores roll and pitch, so this only corrects TF.

Co-Authored-By: Claude Opus 5.5 <noreply@anthropic.com>
Claude-Session: https://claude.ai/code/session_014KtF8zZNgvjM3Zu3cmQvHV

* fix(hardware): time the wheel velocity state on MCU frame stamps

Ticks only advance once per ~50 Hz WHEEL_FEEDBACK frame, while the host
period jitters between 5 and 22 ms. Differentiate over the frames' own
timestamps instead of summed host periods, so the velocity state follows
MCU time and can drive diff_drive's odometry (see the next commit).

Co-Authored-By: Claude Opus 5.5 <noreply@anthropic.com>
Claude-Session: https://claude.ai/code/session_013RrhTFzbyUMRCdxoeaE7V3

* fix(bringup): take odometry from the wheel velocity state

With position feedback, diff_drive divided the 50 Hz tick steps by its
jittery 100 Hz period, so the odom twist read ~5.6 % high and the EKF,
which fuses that twist, put /odom distances 4.4-5.0 % long against lidar
truth. From the MCU-timed velocity state the error is 0.5-2.2 %.

Also stop within 0.5 s when the command stream dies (was 5 s) and shorten
the twist rolling window, since the velocity state is already filtered.

Co-Authored-By: Claude Opus 5.5 <noreply@anthropic.com>
Claude-Session: https://claude.ai/code/session_013RrhTFzbyUMRCdxoeaE7V3

* feat(hardware): default the wheel PID to kp=1.5 ki=3

Live sweep on the floor (in-place spin steps 0.04-0.19 m/s per wheel and
a 0.03-0.05 m/s set, two repeats per gain): against kp=1 ki=2, overshoot
drops from 6.0 to 5.4 %, mid-speed steady-state error from 3.1 to 1.7 %,
low-speed error from 6.7 to 3.9 % and left/right mismatch from 1.2 to
0.4 %, and the wheels settle by the end of the setpoint ramp. kp=2 is only
marginally better; kp=1.5 keeps a 3x margin to the kp=5 oscillation.

Co-Authored-By: Claude Opus 5.5 <noreply@anthropic.com>
Claude-Session: https://claude.ai/code/session_013RrhTFzbyUMRCdxoeaE7V3

* feat(scripts): add the base benchmark harness

bench.py drives tests in a sidecar container (run.sh, data in
~/kestrel_bench) with a geofence, a lidar obstacle guard, stall and
power-dropout watchdogs, and lidar-ICP ground truth. analyze.py turns the
recordings into wheel-loop, latency and odometry metrics, and
pid_summary.py scores a live PID sweep.

Co-Authored-By: Claude Opus 5.5 <noreply@anthropic.com>
Claude-Session: https://claude.ai/code/session_013RrhTFzbyUMRCdxoeaE7V3

* silence the timed out ros2 controller logs

* feat(docker): pin CycloneDDS to WiFi with discovery-only multicast

Without a config, Cyclone binds eth0 whenever the cable is plugged in at
boot, so the robot drops off the graph once it is pulled. Pin DDS to
wlan0 (CYCLONE_IFACE=eth0 for a tethered session) and keep multicast to
SPDP discovery: WiFi sends multicast at the lowest basic rate without
retries, so user data stays unicast even with several remote readers.

Co-Authored-By: Claude Opus 5.5 <noreply@anthropic.com>

* feat(docker): restart the robot bringup unless stopped

Bring the robot stack back up after a reboot or a crash without a manual
docker compose up.

Co-Authored-By: Claude Opus 5.5 <noreply@anthropic.com>

* feat: add the ultra-base-esp32s3 firmware as a submodule

Track the base MCU firmware next to the host stack that talks to it, so a
host commit pins the firmware revision it was tested with.

Co-Authored-By: Claude Opus 5.5 <noreply@anthropic.com>

* feat(scripts): add a WiFi watchdog timer

One WPA handshake timeout fails the profile with no-secrets on the
headless Jetson, and NetworkManager then blocks its autoconnect. Re-up
it every 30 s while wlan0 is disconnected and the SSID is in range.

Co-Authored-By: Claude Opus 5.5 <noreply@anthropic.com>

* feat(description): reverse the base, sensors now at the rear

Rotate the lidar, IMU and ultrasonic mounts 180 deg about z
(x,y -> -x,-y, yaw + pi) so the old front is the new rear.

Co-Authored-By: Claude Opus 5.5 <noreply@anthropic.com>
Claude-Session: https://claude.ai/code/session_01UEzrzT2v2Gej1u4iKEhmYT

* fix(hardware): harden runtime tuning, gpio casts and wheel feedback

- Seed the tuning gpio commands in on_activate so a deactivate/activate
  cycle can't resend zero PID gains or a zero watchdog timeout.
- Ignore non-finite gpio commands and clamp before every integer cast.
- Wait only 20 ms for runtime retune ACKs so write() can't stall 3 s.
- Zero the measured wheel speed when WHEEL_FEEDBACK frames stop for
  0.5 s, and reseed the speed window when they resume.

Co-Authored-By: Claude Opus 5.5 <noreply@anthropic.com>

* fix(bringup): forward use_sim_time to the EKF and wrap a long comment

Co-Authored-By: Claude Opus 5.5 <noreply@anthropic.com>

* fix(scripts): fix bench lint and review findings

- Apply ruff format/check fixes (E741, F841, E731).
- Arm the joint_states staleness check only after the first message.
- Stop the executor before dumping the recording.
- Accept analyze.py output without the entrypoint banner.
- Pass run.sh arguments through without re-splitting them.

Co-Authored-By: Claude Opus 5.5 <noreply@anthropic.com>

* ci: skip the private firmware submodule on recursive clones

CI's GITHUB_TOKEN can't read the private ultra-base-esp32s3 repo, so
recursive checkouts failed. Fetch it explicitly with:
  git submodule update --init --checkout ultra-base-esp32s3

Co-Authored-By: Claude Opus 5.5 <noreply@anthropic.com>

* chore: default the RoboAuto serial port to /dev/ttyACM0

Co-Authored-By: Claude Opus 5.5 <noreply@anthropic.com>

* refactor: rename RoboAuto to Kestrel

Rename the transport class/files, gpio groups (kestrel_pid,
kestrel_watchdog), the tuning controller and the udev rule. The rule now
matches the base on its USB vendor/product ID only and drops the unused
symlink.

Co-Authored-By: Claude Opus 5.5 <noreply@anthropic.com>

* chore: rename RoboLabs to Ultra

Co-Authored-By: Claude Opus 5.5 <noreply@anthropic.com>

---------

Co-authored-by: Claude Opus 5.5 <noreply@anthropic.com>

File: my_diffbot_description/urdf/my_diffbot.urdf.xacro (robot description, xacro)
@@ -5,9 +5,8 @@
   <xacro:arg name="sim_gazebo" default="false" />
   <xacro:arg name="use_mock_hardware" default="false" />
-  <xacro:arg name="use_ultrasonic" default="false" />
-  <xacro:arg name="serial_port" default="/dev/ttyUSB0" />
-  <xacro:arg name="baud_rate" default="57600" />
-  <xacro:arg name="encoder_counts_per_revolution" default="500" />
-  <xacro:arg name="timeout_ms" default="1000" />
+  <xacro:arg name="serial_port" default="/dev/ttyACM0" />
+  <xacro:arg name="baud_rate" default="115200" />
+  <xacro:arg name="encoder_counts_per_revolution" default="515" />
+  <xacro:arg name="timeout_ms" default="20" />
   <!-- Import my_diffbot description -->
   <xacro:include filename="$(find my_diffbot_description)/urdf/my_diffbot_description.xacro" />
@@ -23,5 +22,4 @@
     name="My_diffbot"
     mock_hardware="$(arg use_mock_hardware)"
-    use_ultrasonic="$(arg use_ultrasonic)"
     serial_port="$(arg serial_port)" baud_rate="$(arg baud_rate)"
     encoder_counts_per_revolution="$(arg encoder_counts_per_revolution)"

File: my_diffbot_description/urdf/my_diffbot_description.xacro (robot description, xacro)
@@ -10,18 +10,19 @@
   <xacro:property name="wheel_mass" value="0.3" /> <!-- arbitrary value for wheel mass -->
   <xacro:property name="wheel_len" value="0.025" />
-  <xacro:property name="wheel_radius" value="0.031" />
+  <xacro:property name="wheel_radius" value="0.03" />
+  <xacro:property name="wheel_separation" value="0.255" />  <!-- wheel centre to centre -->
   <xacro:property name="caster_wheel_mass" value="0.1" /> <!-- arbitrary value for caster wheel mass -->
   <xacro:property name="caster_wheel_radius" value="0.015" />
-  <xacro:property name="z_offset" value="-${base_height/2}" /> <!-- Space btw top of beam and the each joint -->
-  <!-- Base Link -->
+  <xacro:property name="chassis_z" value="0.03" /> <!-- chassis bottom above the axle -->
+  <!-- Base Link: base_link is the axle centre, midway between the wheels -->
   <link name="base_footprint"/>
   <joint name="footprint_joint" type="fixed">
     <parent link="base_footprint"/>
     <child link="${prefix}base_link"/>
-    <origin xyz="0.0 0.0 0.05" rpy="0.0 0.0 0.0"/>
+    <origin xyz="0.0 0.0 ${wheel_radius}" rpy="0.0 0.0 0.0"/>
   </joint>
   <link name="${prefix}base_link">
     <collision>
-      <origin xyz="0 0 ${base_height/2}" rpy="0 0 0"/>
+      <origin xyz="0 0 ${chassis_z + base_height/2}" rpy="0 0 0"/>
       <geometry>
         <cylinder radius="0.15" length="0.06"/>
@@ -29,5 +30,5 @@
     </collision>
     <visual>
-      <origin xyz="0 0 ${base_height/2}" rpy="0 0 0"/>
+      <origin xyz="0 0 ${chassis_z + base_height/2}" rpy="0 0 0"/>
       <geometry>
         <cylinder radius="0.15" length="0.06"/>
@@ -35,5 +36,5 @@
     </visual>
     <inertial>
-      <origin xyz="0 0 0" rpy="0 0 0"/>
+      <origin xyz="0 0 ${chassis_z + base_height/2}" rpy="0 0 0"/>
       <mass value="${base_mass}"/>
       <inertia
@@ -43,9 +44,11 @@
       </inertial>
     </link>
-    <!-- LIDAR -->
+    <!-- LIDAR: x, y and yaw are the LD06 scan frame, fitted from scan matching over
+         straight drives and in-place turns (yaw -86.5 deg, not -90), then rotated 180 deg
+         about z when the base was reversed (old front is now the rear) -->
     <joint name="lidar_joint" type="fixed">
       <parent link="${prefix}base_link"/>
       <child link="${prefix}lidar_link"/>
-      <origin xyz="-0.06 0.0 0.14" rpy="0.0 0.0 1.57"/>
+      <origin xyz="-0.110 0.023 0.14" rpy="0.0 0.0 ${-1.510 + PI}"/>
     </joint>
     <link name="${prefix}lidar_link">
@@ -61,5 +64,5 @@
       <parent link="${prefix}base_link"/>
       <child link="${prefix}ultrasonic_link"/>
-      <origin xyz="-0.12 0.0 0.0" rpy="0.0 0.0 -3.14"/>
+      <origin xyz="0.12 0.0 ${chassis_z}" rpy="0.0 0.0 0.0"/>
     </joint>
     <link name="${prefix}ultrasonic_link">
@@ -71,9 +74,11 @@
       </visual>
     </link>
-    <!-- IMU -->
+    <!-- IMU: the firmware remap leaves /imu/data x pointing to the old rear, which is the
+         front since the base was reversed (accel while driving).
+         The board is pitched 5.9 deg (calibrated accel at rest; the lidar plane is level). -->
     <joint name="imu_joint" type="fixed">
       <parent link="${prefix}base_link"/>
       <child link="${prefix}imu_link"/>
-      <origin xyz="0.0 0.025 0.065" rpy="0.0 0.0 0.0"/>
+      <origin xyz="-0.04 0.0 0.045" rpy="0.0 -0.103 0.0"/>
     </joint>
     <link name="${prefix}imu_link">
@@ -89,5 +94,5 @@
       <parent link="${prefix}base_link"/>
       <child link="${prefix}left_wheel"/>
-      <origin xyz="0 -${base_width/2} ${z_offset}" rpy="0 0 0"/>
+      <origin xyz="0 ${wheel_separation/2} 0" rpy="0 0 0"/>
       <axis xyz="0 1 0"/>
       <dynamics damping="0.2"/>
@@ -120,5 +125,5 @@
       <parent link="${prefix}base_link"/>
       <child link="${prefix}right_wheel"/>
-      <origin xyz="0 ${base_width/2} ${z_offset}" rpy="0 0 0"/>
+      <origin xyz="0 -${wheel_separation/2} 0" rpy="0 0 0"/>
       <axis xyz="0 1 0"/>
       <dynamics damping="0.2"/>
@@ -151,5 +156,5 @@
       <parent link="${prefix}base_link"/>
       <child link="${prefix}caster_frontal_wheel"/>
-      <origin xyz="${base_width/2 - caster_wheel_radius} 0 ${z_offset}" rpy="0 0 0"/>
+      <origin xyz="${base_width/2 - caster_wheel_radius} 0 ${caster_wheel_radius - wheel_radius}" rpy="0 0 0"/>
     </joint>
     <!-- caster frontal wheel Link -->
@@ -179,5 +184,5 @@
       <parent link="${prefix}base_link"/>
       <child link="${prefix}caster_rear_wheel"/>
-      <origin xyz="${-base_width/2 + caster_wheel_radius} 0 ${z_offset}" rpy="0 0 0"/>
+      <origin xyz="${-base_width/2 + caster_wheel_radius} 0 ${caster_wheel_radius - wheel_radius}" rpy="0 0 0"/>
     </joint>
     <!-- caster rear wheel Link -->
